Commit message: estabilidad en seguimiento

File: install/skycam_description/share/skycam_description/urdf/ball.xacro (robot description, xacro)
@@ -12,6 +12,6 @@
         <sphere radius="0.11"/>
       </geometry>
-      <material name="white">
-        <color rgba="1.0 1.0 1.0 1.0"/>
+      <material name="orange">
+        <color rgba="1.0 0.5 0.0 1.0"/>
       </material>
     </visual>
@@ -24,5 +24,5 @@
   </link>
   <gazebo reference="base_link">
-    <material>Gazebo/White</material>
+    <material>Gazebo/Orange</material>
     <mu1>0.0</mu1>
     <mu2>0.0</mu2>

File: install/skycam_description/share/skycam_description/urdf/simple_sphere.xacro (robot description, xacro)
@@ -13,6 +13,6 @@
         <sphere radius="${radius}"/>
       </geometry>
-      <material name="blue">
-        <color rgba="0 0 1 1"/>
+      <material name="Orange">
+        <color rgba="1.0 0.5 0.0 1.0"/>
       </material>
     </visual>
@@ -35,7 +35,12 @@
   </link>
   <gazebo reference="base_link">
-    <material>Gazebo/Blue</material>
+    <material>Gazebo/Orange</material>
+    <visual>
+      <material>
+        <ambient>1.0 0.5 0.0 1.0</ambient>
+        <diffuse>1.0 0.5 0.0 1.0</diffuse>
+      </material>
+    </visual>
   </gazebo>
-  <gazebo>
     <plugin name="sphere_odom" filename="libgazebo_ros_p3d.so">
       <ros>

File: install/skycam_description/share/skycam_description/urdf/skycam_gazebo.xacro (robot description, xacro)
@@ -75,5 +75,5 @@
   <gazebo reference="camera_link">
     <sensor type="camera" name="skycam_camera">
-      <update_rate>60.0</update_rate>
+      <update_rate>30.0</update_rate>
       <camera name="head">
         <horizontal_fov>1.3962634</horizontal_fov>
